File: Eagle/Synth_pcb_v1/Synth_pcb_v1.sch (EAGLE design)
At the start: 28 parts, among them IC3 LM358N, T1 BC547, T2 BC547, X1 MAB5SH

Commit message: Complete schematics, ready to start designing PCB.
Parts:
- added C10: 10nF, capacitor-wima:C2,5-3
- added C4, C6, C8: 220nF, capacitor-wima:C2,5-3
- added C5, C7: 22uF, capacitor-wima:C2,5-3
- added C9: 100nF, capacitor-wima:C2,5-3
- added IC4, IC5, IC6: LM358N, linear:LM358N
- added JP6, JP8, JP9: (no value), pinhead:PINHD-1X2
- added JP7: (no value), pinhead:PINHD-1X3
- added R11, R19, R27: 4.7k, resistor-power:RAC01
- added R12, R14, R15, R18, R20, R22, R23, R26, R28, R33, R34, R37: 1k, resistor-power:RAC01
- added R13, R16, R17, R21, R24, R25, R29, R30, R31, R32, R36, R6: 10k, resistor-power:RAC01
- added R35: NC, resistor-power:RAC01
- added T3, T4, T5, T6: BC547, transistor:BC547
- C2: value 10uF -> 22uF
- R10: value 220k -> 1k
- R8: value 470 -> 1k
Connections:
- removed net GND1: JP4.1
- removed net N$17: IC2.IN
- removed net N$18: IC3A.OUT, JP4.2
- removed net N$19: R7.1
- removed net N$2: D2.A
- removed net N$20: R5.2
- removed net N$23: R10.2, T1.C
- removed net N$9: OK1.VO, R2.1
- removed net TRIGGER_SAW: ARDUINO_NANO1.D5
- new net AMP1_OUT: IC6A.OUT, JP4.2
- new net AMP2_OUT: IC6B.OUT, JP7.2
- new net AUDIO_IN: ARDUINO_NANO1.A2
- new net HPF_OUT: C10.1, JP6.2
- new net LPF_OUT: IC6A.+IN, JP5.2
- new net N$28: R13.2
- new net N$29: C5.1, R14.2, R15.1, T3.C
- new net N$30: C5.2, T4.C
- new net N$33: C6.1, IC4A.-IN, R15.2, R17.2
- new net N$34: C6.2, IC4A.OUT, R17.1, R18.2
- new net N$35: IC4B.-IN, R18.1, R19.1, R20.2
- new net N$36: R13.1, T3.B
- new net N$37: R16.1, T4.B
- new net N$38: R22.1
- new net N$39: R21.2
- new net N$40: C7.1, R22.2, R23.1, T5.C
- new net N$41: C7.2, T6.C
- new net N$44: C8.1, IC5A.-IN, R23.2, R25.2
- new net N$45: C8.2, IC5A.OUT, R25.1, R26.2
- new net N$46: IC5B.-IN, R26.1, R27.1, R28.2
- new net N$47: R21.1, T5.B
- new net N$48: R24.1, T6.B
- new net N$49: R29.2
- new net N$50: R30.2
- new net N$51: R31.2
- new net N$54: R16.2
- new net N$55: JP8.2
- new net N$56: C10.2
- new net N$57: IC6B.-IN, JP7.3, R34.2
- new net N$58: IC6A.-IN, JP4.3, R33.2
- new net N$59: C9.2, JP5.3
- new net N$60: IC6B.+IN
- new net N$61: JP9.2
- new net N$62: R24.2
- new net N$63: JP9.1, R35.2
- new net N$65: R37.2
- new net N$66: R36.2, R37.1
- new net OUT_OSC2: IC4B.OUT, R20.1
- new net OUT_OSC3: IC5B.OUT, R28.1
- new net OUT_WAV: R29.1, R30.1, R31.1
- new net TRIGGER_TRI: ARDUINO_NANO1.D5, R9.2
- net 0V_IN: now also D2.A, IC3P.V-, IC4P.V-, IC5P.V-, IC6P.V-
- net CONTROL_OSC1: now also R5.2
- net GND: now also ARDUINO_NANO1.AREF, C9.1, IC3A.+IN, IC3B.+IN, IC4A.+IN, IC4B.+IN, IC5A.+IN, IC5B.+IN, JP8.1, OK1.GND, R3.1, R32.1, R33.1, R34.1, R35.1, R36.1, T3.E, T4.E, T5.E, T6.E; no longer IC3A.-IN
- net GND2: now also JP6.1, R32.2; no longer JP5.1
- net MIDI_IN: now also OK1.VO, R2.1
- net N$16: now also C4.1, IC3A.-IN, R6.2, R8.2; no longer IC3A.+IN
- net N$24: now also T1.C; no longer R10.1
- net N$25: now also C4.2, IC3A.OUT, R10.2, R6.1; no longer JP4.3
- net N$26: now also IC3B.-IN, R10.1, R11.1, R12.2; no longer JP5.2
- net N$27: now also R14.1; no longer JP5.3
- net N$8: now also JP5.1; no longer OK1.GND, R3.1
- net OUT_OSC1: now also IC3B.OUT, R12.1; no longer R8.2
- net REG_5V: now also IC3P.V+, IC4P.V+, IC5P.V+, IC6P.V+, R11.2, R19.2, R27.2, R7.1
- net V+: now also IC2.IN
Other:
- note added: "AMP GAIN"
- note added: "AUDIO IN"
- note added: "AUDIO OUT"
- note added: "LOW-PASS FILTER"
- note added: "MIXER"
- note added: "Mixer"
- note added: "OSCILLATOR 1"
- note added: "OSCILLATOR 2"
- note added: "OSCILLATOR 3"
- note added: "VOLUME OUT"
- note removed: "10k POT GAIN"
- note removed: "1k POT - OFFSET"
- moved on the sheet: C2, IC3A, JP4, JP5, R10, R5, R7, R8, R9, SV2, T1, T2

Commit message: First iteration on PCB design, schematic revised
Parts:
- added JP10: (no value), pinhead:PINHD-1X3
- added R38: 1k, rcl:R-EU_0204/7
- R1, R10, R11, R12, R13, R14, R15, R16, R17, R18, R19, R2, R20, R21, R22, R23, R24, R25, R26, R27, R28, R29, R3, R30, R31, R32, R33, R34, R35, R36, R37, R4, R5, R6, R7, R8, R9: device resistor-power:RAC01 -> rcl:R-EU_0204/7
Connections:
- removed net N$10: OK1.VCC, R2.2
- removed net N$12: JP1.2
- removed net N$14: R4.1
- removed net N$15: JP3.2
- removed net N$27: R14.1
- removed net N$28: R13.2
- removed net N$3: C1.2, IC1.GND
- removed net N$38: R22.1
- removed net N$39: R21.2
- removed net N$4: JP2.1
- removed net N$49: R29.2
- removed net N$50: R30.2
- removed net N$51: R31.2
- removed net N$54: R16.2
- removed net N$55: JP8.2
- removed net N$56: C10.2
- removed net N$60: IC6B.+IN
- removed net N$61: JP9.2
- removed net N$62: R24.2
- removed net N$65: R37.2
- removed net N$66: R36.2, R37.1
- removed net N$8: JP5.1
- new net N$2: IC6B.OUT, JP7.2, R38.2
- new net PWR: JP10.3, SV2.3
- net 0V_IN: now also JP10.1
- net 12V_IN: now also C1.2, IC1.GND, JP10.2; no longer SV2.3
- net 5V: now also JP2.1, OK1.VCC, R2.2, R4.1
- net AMP1_OUT: now also C10.2
- net AMP2_OUT: now also JP8.2, JP9.2, R37.2, R38.1; no longer IC6B.OUT, JP7.2
- net AUDIO_IN: now also R36.2, R37.1
- net CONTROL_OSC2: now also R13.2
- net CONTROL_OSC3: now also R21.2
- net HPF_OUT: now also IC6B.+IN
- net IN_0: now also JP1.2
- net IN_1: now also JP3.2
- net OUT_OSC1: now also R29.2
- net OUT_OSC2: now also R30.2
- net OUT_OSC3: now also R31.2
- net OUT_WAV: now also JP5.1
- net REG_5V: now also R14.1, R22.1
- net TRIGGER_TRI: now also R16.2, R24.2
Other:
- note added: "AUDIO MONITOR"
- note added: "SWITCH"
- note removed: "AUDIO IN"

Commit message: Most of the PCB is routed. Revision is needed
Connections:
- net CONTROL_OSC1: now also ARDUINO_NANO1.D8; no longer ARDUINO_NANO1.D6
- net CONTROL_OSC3: now also ARDUINO_NANO1.D6; no longer ARDUINO_NANO1.D8
Changed lines of the file:
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@@
 <net name="CONTROL_OSC1" class="0">
-<segment>
-<pinref part="ARDUINO_NANO1" gate="G$1" pin="D6"/>
-<wire x1="71.12" y1="58.42" x2="76.2" y2="55.88" width="0.1524" layer="91"/>
-<label x="76.2" y="55.88" size="1.778" layer="95" xref="yes"/>
-<junction x="71.12" y="58.42"/>
-</segment>
 <segment>
 <pinref part="R5" gate="G$1" pin="2"/>
 <wire x1="162.56" y1="63.5" x2="154.94" y2="63.5" width="0.1524" layer="91"/>
 <label x="154.94" y="63.5" size="1.778" layer="95" rot="R180" xref="yes"/>
+</segment>
+<segment>
+<pinref part="ARDUINO_NANO1" gate="G$1" pin="D8"/>
+<wire x1="71.12" y1="63.5" x2="76.2" y2="66.04" width="0.1524" layer="91"/>
+<label x="76.2" y="66.04" size="1.778" layer="95" xref="yes"/>
+<label x="299.72" y="60.96" size="1.778" layer="95" rot="R180" xref="yes"/>
+<junction x="71.12" y="63.5"/>
 </segment>
 </net>
@@
 <net name="CONTROL_OSC3" class="0">
 <segment>
-<pinref part="ARDUINO_NANO1" gate="G$1" pin="D8"/>
-<wire x1="71.12" y1="63.5" x2="76.2" y2="66.04" width="0.1524" layer="91"/>
-<label x="76.2" y="66.04" size="1.778" layer="95" xref="yes"/>
-<label x="299.72" y="60.96" size="1.778" layer="95" rot="R180" xref="yes"/>
-<junction x="71.12" y="63.5"/>
-</segment>
-<segment>
 <wire x1="299.72" y1="60.96" x2="304.8" y2="60.96" width="0.1524" layer="91"/>
 <pinref part="R21" gate="G$1" pin="2"/>
 <junction x="304.8" y="60.96"/>
 </segment>
+<segment>
+<pinref part="ARDUINO_NANO1" gate="G$1" pin="D6"/>
+<wire x1="71.12" y1="58.42" x2="76.2" y2="55.88" width="0.1524" layer="91"/>
+<label x="76.2" y="55.88" size="1.778" layer="95" xref="yes"/>
+<junction x="71.12" y="58.42"/>
+</segment>
 </net>

Commit message: PCB routing complete, ready for revision.
Parts:
- C10: value 10nF -> 220nF
- C2: value 22uF -> 220uF
- C3: value 220uF -> 22uF
- C4: value 220nF -> 22uF
- C5: value 22uF -> 220nF
- C7: value 22uF -> 100nF
- C8: value 220nF -> 10nF
- C9: value 100nF -> 22uF
- D1: value 1N4004 -> ZY; device diode:1N4004 -> diode:ZY
- D2: value ZY -> 1N4004; device diode:ZY -> diode:1N4004
- JP2: device pinhead:PINHD-1X4 -> pinhead:PINHD-1X2
- JP3: device pinhead:PINHD-1X2 -> pinhead:PINHD-1X4
- JP5, JP7: device pinhead:PINHD-1X3 -> pinhead:PINHD-1X2
- JP8, JP9: device pinhead:PINHD-1X2 -> pinhead:PINHD-1X3
- R11: value 4.7k -> 1k
- R12, R18, R26, R34, R7, R8: value 1k -> 10k
- R16, R17, R3, R30, R32, R36, R6: value 10k -> 1k
- R19, R27: value 4.7k -> 10k
- R2: value 470 -> NC
- R20: value 1k -> 4.7k
- R21: value 10k -> 4.7k
- R35: value NC -> 4.7k
- R4: value 1k -> 470
- renumbered SV2 to SV1
Connections:
- removed net N$21 (its old number): R5.1, T1.B
- new net N$22: R13.1, T4.B
- net 0V_IN: now also D1.A, JP1.1; no longer D2.A, JP10.1
- net 12V_IN: now also JP1.2; no longer JP10.2
- net 5V: now also JP3.1, R3.1, R4.2; no longer JP2.1, R2.2, R4.1
- net AMP1_OUT: now also C8.2, JP10.2; no longer C10.2, JP4.2
- net AMP2_OUT: now also JP2.2, JP5.2, R33.1, R6.2; no longer JP8.2, JP9.2, R37.2, R38.1
- net AUDIO_IN: now also R6.1, R7.2; no longer R36.2, R37.1
- net CONTROL_OSC1: now also R9.2; no longer R5.2
- net CONTROL_OSC2: now also R8.2; no longer R13.2
- net CONTROL_OSC3: now also R24.2; no longer R21.2
- net GND: now also C2.2, C7.1, D1.C, JP2.1, JP3.2, JP4.1, JP6.1, R2.1, R31.1, R37.1, R38.1, R5.1, R7.1; no longer C3.2, C9.1, D2.C, JP1.1, JP2.2, JP3.1, JP8.1, R3.1, R32.1, R33.1, R34.1, R35.1, R36.1
- net GND2: now also JP7.1, R31.2; no longer JP6.1, R32.2
- net HPF_OUT: now also C8.1, JP7.2; no longer C10.1, JP6.2
- net IN_0: now also JP4.2; no longer JP1.2
- net IN_1: now also JP6.2; no longer JP3.2
- net LPF_OUT: now also JP8.2; no longer JP5.2
- net MIDI_IN: now also R4.1; no longer R2.1
- net N$1: now also D2.A; no longer D1.A
- net N$11: now also C4.2, T4.C; no longer C2.2, T2.C
- net N$13: now also JP4.3, R3.2; no longer JP1.3, R4.2
- net N$16: now also C6.1, IC4A.-IN, R14.2, R19.2; no longer C4.1, IC3A.-IN, R6.2, R8.2
- net N$2: now also JP9.2, R33.2; no longer JP7.2, R38.2
- net N$24: now also C4.1, R11.2, R14.1, T2.C; no longer C2.1, R7.2, R8.1, T1.C
- net N$25: now also C6.2, IC4A.OUT, R19.1, R23.2; no longer C4.2, IC3A.OUT, R10.2, R6.1
- net N$26: now also IC4B.-IN, R17.2, R21.1, R23.1; no longer IC3B.-IN, R10.1, R11.1, R12.2
- net N$29: now also C3.1, R10.2, T1.C; no longer C5.1, R14.2, T3.C
- net N$30: now also C3.2, T3.C; no longer C5.2, T4.C
- net N$33: now also C5.1, IC3A.-IN, R18.2; no longer C6.1, IC4A.-IN, R17.2
- net N$34: now also C5.2, IC3A.OUT, R18.1, R22.2; no longer C6.2, IC4A.OUT, R17.1, R18.2
- net N$35: now also IC3B.-IN, R16.2, R20.1, R22.1; no longer IC4B.-IN, R18.1, R19.1, R20.2
- net N$36: now also R8.1, T1.B; no longer R13.1, T3.B
- net N$37: now also R12.1, T3.B; no longer R16.1, T4.B
- net N$40: now also C9.1, R28.2, R30.1; no longer C7.1, R22.2, R23.1
- net N$41: now also C9.2; no longer C7.2
- net N$44: now also C10.1, R30.2, R34.2; no longer C8.1, R23.2, R25.2
- net N$45: now also C10.2, R34.1, R36.2; no longer C8.2, R25.1, R26.2
- net N$46: now also R32.2, R35.1, R36.1; no longer R26.1, R27.1, R28.2
- net N$47: now also R24.1; no longer R21.1
- net N$48: now also R29.1; no longer R24.1
- net N$5: now also D2.C; no longer D1.C
- net N$57: now also JP9.3, R38.2; no longer JP7.3, R34.2
- net N$58: now also JP10.3, R37.2; no longer JP4.3, R33.2
- net N$59: now also C7.2, JP8.3; no longer C9.2, JP5.3
- net N$63: now also JP5.1, R2.2; no longer JP9.1, R35.2
- net N$7: now also R5.2; no longer R3.2
- net OUT_OSC1: now also IC4B.OUT, R17.1, R27.2; no longer IC3B.OUT, R12.1, R29.2
- net OUT_OSC2: now also IC3B.OUT, R16.1, R26.2; no longer IC4B.OUT, R20.1, R30.2
- net OUT_OSC3: now also R25.2, R32.1; no longer R28.1, R31.2
- net OUT_WAV: now also JP8.1, R25.1, R26.1, R27.1; no longer JP5.1, R29.1, R30.1, R31.1
- net PWR: now also JP1.3; no longer JP10.3
- net REG_5V: now also C2.1, R10.1, R11.1, R20.2, R21.2, R28.1, R35.2; no longer C3.1, R11.2, R14.1, R19.2, R22.1, R27.2, R7.1
- net SCL: now also JP3.3; no longer JP2.3
- net SDA: now also JP3.4; no longer JP2.4
- net TRIGGER_TRI: now also R12.2, R13.2, R29.2; no longer R16.2, R24.2, R9.2
Other:
- moved on the sheet: C10, C2, C3, C4, C5, C6, C7, C8, C9, IC3A, IC3B, IC4A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
