File: Eagle/Synth_pcb_v2/Synth_pcb_v2.sch (EAGLE design)
At the start: 76 parts, among them IC3 LM358N, IC4 LM358N, IC5 LM358N, IC6 LM358N, T1 BC547, T2 BC547, T3 BC547, T4 BC547, T5 BC547, T6 BC547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

Commit message: PCB complete and sent to be manufactured
Parts:
- C10: value 220nF -> 10nF
- C7: value 100nF -> 22uF
- C8: value 10nF -> 100nF
- C9: value 22uF -> 220nF
- IC1: device v-reg:79XXS -> v-reg:78XXS
- IC2: device v-reg:78XXS -> v-reg:79XXS
- JP10, JP4, JP8, JP9: device pinhead:PINHD-1X3 -> pinhead:PINHD-1X2
- JP2: device pinhead:PINHD-1X2 -> pinhead:PINHD-1X4
- JP3: device pinhead:PINHD-1X4 -> pinhead:PINHD-1X3
- JP6: device pinhead:PINHD-1X2 -> pinhead:PINHD-1X3
- R1: value 220 -> 1k
- R14, R15, R16, R17, R22, R33, R38: value 1k -> 10k
- R18: value 10k -> 470
- R19: value 10k -> 220
- R2: value NC -> 1k
- R20, R35: value 4.7k -> 10k
- R21: value 4.7k -> 1k
- R26: value 10k -> 4.7k
- R27, R29, R5, R7, R8, R9: value 10k -> 1k
- R36: value 1k -> NC
- R4: value 470 -> 4.7k
- R6: value 1k -> 4.7k
- X1: device con-hirschmann:MAB5SH -> con-hirschmann_alt:MAB5SH
Connections:
- net 0V_IN: now also IC2.IN; no longer IC1.IN
- net 12V_IN: now also IC2.GND; no longer IC1.GND
- net 5V: now also JP2.1, R18.2; no longer JP3.1, R4.2
- net AMP1_OUT: now also JP10.1, JP6.1; no longer C8.2, JP10.2
- net AMP2_OUT: now also JP7.2, JP8.2, R30.1, R32.2; no longer JP2.2, JP5.2, R33.1, R6.2
- net AUDIO_IN: now also R32.1, R35.2; no longer R6.1, R7.2
- net CONTROL_OSC1: now also R12.2; no longer R9.2
- net CONTROL_OSC2: now also R13.2; no longer R8.2
- net CONTROL_OSC3: now also R31.2; no longer R24.2
- net GND: now also C8.1, IC1.GND, JP2.2, JP3.1, JP7.1, R23.1, R24.1, R35.1, R36.1; no longer C7.1, IC2.GND, JP2.1, JP3.2, JP6.1, R2.1, R31.1, R5.1, R7.1
- net GND2: now also JP9.1, R38.2; no longer JP7.1, R31.2
- net HPF_OUT: now also C10.1, JP9.2; no longer C8.1, JP7.2
- net IN_0: now also JP3.2; no longer JP4.2
- net IN_1: now also JP4.2; no longer JP6.2
- net LPF_OUT: now also C10.2, JP6.2; no longer IC6A.+IN, JP8.2
- net MIDI_IN: now also R18.1; no longer R4.1
- net N$13: now also JP3.3; no longer JP4.3
- net N$16: now also C5.1, IC3A.-IN, R10.2, R15.2; no longer C6.1, IC4A.-IN, R14.2, R19.2
- net N$2: now also JP5.1, R30.2; no longer JP9.2, R33.2
- net N$21: now also R12.1, T1.B; no longer R9.1, T2.B
- net N$22: now also R14.1, T3.B; no longer R13.1, T4.B
- net N$24: now also C3.1, R10.1, R8.2, T1.C; no longer C4.1, R11.2, R14.1, T2.C
- net N$25: now also C5.2, IC3A.OUT, R15.1, R5.2; no longer C6.2, IC4A.OUT, R19.1, R23.2
- net N$26: now also IC3B.-IN, R1.2, R4.1, R5.1; no longer IC4B.-IN, R17.2, R21.1, R23.1
- net N$29: now also C4.1, R11.1, R9.2, T2.C; no longer C3.1, R10.2, R15.1, T1.C
- net N$33: now also C6.1, IC4A.-IN, R11.2, R17.2; no longer C5.1, IC3A.-IN, R15.2, R18.2
- net N$34: now also C6.2, IC4A.OUT, R17.1, R7.2; no longer C5.2, IC3A.OUT, R18.1, R22.2
- net N$35: now also IC4B.-IN, R2.2, R6.1, R7.1; no longer IC3B.-IN, R16.2, R20.1, R22.1
- net N$36: now also R13.1, T2.B; no longer R8.1, T1.B
- net N$37: now also R16.1, T4.B; no longer R12.1, T3.B
- net N$40: now also C7.1, R29.1; no longer C9.1, R30.1
- net N$41: now also C7.2; no longer C9.2
- net N$44: now also C9.1, R29.2; no longer C10.1, R30.2
- net N$45: now also C9.2, R27.2; no longer C10.2, R36.2
- net N$46: now also R21.2, R26.1, R27.1; no longer R32.2, R35.1, R36.1
- net N$47: now also R31.1; no longer R24.1
- net N$48: now also R33.1; no longer R29.1
- net N$5: now also R19.2; no longer R1.2
- net N$57: now also JP5.2, R23.2; no longer JP9.3, R38.2
- net N$58: now also JP10.2; no longer JP10.3
- net N$59: now also C8.2, JP6.3; no longer C7.2, JP8.3
- net N$6: now also R19.1; no longer R1.1
- net N$63: now also JP8.1, R36.2; no longer JP5.1, R2.2
- net N$7: now also R24.2; no longer R5.2
- net OUT_OSC1: now also IC3B.OUT, R1.1, R20.2; no longer IC4B.OUT, R17.1, R27.2
- net OUT_OSC2: now also IC4B.OUT, R2.1, R22.2; no longer IC3B.OUT, R16.1, R26.2
- net OUT_OSC3: now also R21.1; no longer R32.1
- net OUT_WAV: now also IC6A.+IN, R20.1, R22.1; no longer JP8.1, R26.1, R27.1
- net REG_5V: now also IC1.OUT, R26.2, R4.2, R6.2, R8.1, R9.1; no longer IC2.OUT, R10.1, R11.1, R20.2, R21.2, R35.2
- net SCL: now also JP2.3; no longer JP3.3
- net SDA: now also JP2.4; no longer JP3.4
- net TRIGGER_TRI: now also R14.2, R16.2, R33.2; no longer R12.2, R13.2, R29.2
- net V+: now also IC1.IN, IC2.OUT; no longer IC1.OUT, IC2.IN
Other:
- moved on the sheet: ARDUINO_NANO1, C1, C10, C2, C3, C4, C5, C6, C7, C8, C9, D1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

Commit message: Revision B made on time of manufacturing: corrected power schematic
Parts:
- renumbered ARDUINO_NANO1 to ARDUINO_NANO
Connections:
- removed net PWR: JP1.3, SV1.3
- new net 0V: IC2.IN, JP1.1, SV1.1
- net 0V_IN: now also C1.2, IC2.OUT; no longer C1.1, IC2.IN, JP1.1, SV1.2
- net 12V_IN: now also ARDUINO_NANO.VIN, C1.1, IC1.IN; no longer C1.2
- net V+: now also JP1.3, SV1.2; no longer ARDUINO_NANO.VIN, IC1.IN, IC2.OUT
Other:
- moved on the sheet: C1, IC2
